File: InstrumentBuild/EAGLE/optMotorDriver.sch (EAGLE design)
At the start: 69 parts, among them IC1 A4988ALT1, IC2 LM317L, J1 1X2-3.5MM, J2 1X2-3.5MM, J4 1X2-3.5MM, J5 1X2-3.5MM, J6 1X2-3.5MM, U1 ARDUINOR3-DIMENSION

Commit message: Update schematics and readme for driver board.
Parts:
- removed 3/5V: SOLDERJUMPERNO, SparkFun03_30_09:SOLDERJUMPERNO
- removed APWR: SOLDERJUMPERTRACE, SparkFun03_30_09:SOLDERJUMPERTRACE
- removed C10: .22uF, SparkFun-Capacitors:0.22UF50V-20%,+80%(0603)
- removed C11, C6, C7, C8, C9: .1uf, SparkFun-Capacitors:0.1UF-100V-10%(0603)
- removed C14: 47uF, SparkFun-Capacitors:47UF-50V-20%(ELECT)
- removed D1: B340A-13-F, diode:DIODE-DO-214AC
- removed FID1, FID2: FIDUCIAL1X2, SparkFun-Aesthetics:FIDUCIAL1X2
- removed FRAME1: FRAME-LETTER, SparkFun-Aesthetics:FRAME-LETTER
- removed IC1: A4988ALT1, SparkFun-PowerIC:A4988ALT1
- removed IC2: LM317L, BigEasyDriver_v11:SPARKFUN03_30_09_V_REG_317SOT89SOT89
- removed J4, J5, J6, MOTOR_PWR: 1X2-3.5MM, adafruit:1X2-3.5MM
- removed JP1, JP6: (no value), SparkFun:M02PTH
- removed JP10, JP14, JP15, JP3: (no value), SparkFun:M04PTH
- removed JP11, JP12, JP5: (no value), BigEasyDriver_v11:M04SCREW_LOCK
- removed JP13, JP7: (no value), BigEasyDriver_v11:M023.5MM_LOCK
- removed JP8, JP9: STAND-OFF, SparkFun-7-28-09:STAND-OFF
- removed LOGO1: OSHW_LOGO_FILLX0100-NT, OSHW:OSHW_LOGO_FILLX0100-NT
- removed PWR_LED: YELLOW, SparkFun03_30_09:LED0603
- removed R10, R11, R12, R20: 20K, SparkFun-Resistors:20KOHM1/10W5%(0603)
- removed R13: 8.2K, SparkFun-Resistors:8.2KOHM-1/10W-5%(0603)
- removed R14, R15, R9: 1K, SparkFun-Resistors:1KOHM1/10W1%(0603)
- removed R16: 10K, SparkFun-Electromechanical:TRIMPOT3MM-2
- removed R18, R19: .11, SparkFun-Resistors:0.11OHM1/2W1%(2010)
- removed R7: 330, SparkFun-Resistors:330OHM1/10W1%(0603)
- removed R8: 240, SparkFun-Resistors:240OHM1/10W1%(0603)
- removed S1: (no value), adafruit:40-XX
- removed TP1: TPPAD1-13, testpad:TPPAD1-13
- removed U$2: LOGO-SFENEW, SparkFun:LOGO-SFENEW
- removed U$3, U$4, U$5: PAD, Testing:PAD
- added ACOIL, BCOIL, C3, C4, C5, TRIGGER: 1X2-3.5MM, adafruit:1X2-3.5MM
- added MOTOR: (no value), SparkFun:M04PTH
- added S2: (no value), SparkFun-Switches:MOMENTARY-SWITCH-SPST-2-SMD-5.2MM
- C1: value .1uF -> 1X2-3.5MM; device SparkFun-Capacitors:0.1UF-100V-10%(0603) -> adafruit:1X2-3.5MM
- C2: value 1uF -> 1X2-3.5MM; device SparkFun-Capacitors:1.0UF-16V-10%(0603) -> adafruit:1X2-3.5MM
- J1: value 1X2-3.5MM -> (none); device adafruit:1X2-3.5MM -> Wurth_Elektronik_Electromechanic_Wire_to_Board_Connectors_rev19a:62400821722
- J2: value 1X2-3.5MM -> (none); device adafruit:1X2-3.5MM -> con-jack:DCJ0303
- R1, R2, R3, R4, R5: value 20K -> 10kΩ; device SparkFun-Resistors:20KOHM1/10W5%(0603) -> adafruit:R-US_R1206
- R17: device adafruit:R-US_V234/12 -> adafruit:R-US_R1206
- R6: value 390 -> 10kΩ; device SparkFun-Resistors:390OHM1/10W1%(0603) -> adafruit:R-US_R1206
Connections:
- removed net 5V_ALT: APWR.1, IC2.OUT, IC2.OUT@1, R8.2
- removed net CUR_REF: IC1.REF, R16.WIPER, TP1.TP
- removed net DIR: IC1.DIR, R11.1, R14.2
- removed net GND1: JP17.1, MOTOR_PWR.2
- removed net N$10: IC1.NC@3, U$5.P$1
- removed net N$11: JP17.2, MOTOR_PWR.1
- removed net N$12: J6.1, R17.2, U1.GND1, U1.GND2
- removed net N$17: S1.P, U1.D12
- removed net N$19: IC1.ROSC, R20.1
- removed net N$20: C10.1, IC1.VREG
- removed net N$21: C11.1, IC1.VCP
- removed net N$31: IC1.SENSE2, R18.2
- removed net N$32: IC1.SENSE1, R19.2
- removed net N$4: 3/5V.1, R6.1, R7.2
- removed net N$5: IC1.NC@1, U$3.P$1
- removed net N$9: C6.2, IC1.CP2
- removed net STEP: IC1.STEP, R12.1, R15.2
- removed net V+: C1.1, C11.2, C14.+, C8.1, C9.1, D1.C, IC1.VBB1, IC1.VBB2, IC2.IN
- net COILA+: now also ACOIL.2, MOTOR.4; no longer IC1.OUT1B, J2.2, JP15.4, JP3.4, JP5.4
- net COILA-: now also ACOIL.1, MOTOR.3; no longer IC1.OUT1A, J2.1, JP15.3, JP3.3, JP5.3
- net COILB+: now also BCOIL.1, MOTOR.1; no longer IC1.OUT2B, J1.1, JP15.1, JP3.1, JP5.1
- net COILB-: now also BCOIL.2, MOTOR.2; no longer IC1.OUT2A, J1.2, JP15.2, JP3.2, JP5.2
- net DIR_IN: no longer JP12.4, JP14.4, R14.1
- net ENABLE: no longer IC1.ENABLE, JP13.1, JP6.1, R10.1
- net GND: now also C1.1, C2.1, C3.1, C4.1, C5.1, R1.1, R17.2, R2.1, R3.1, R4.1, R5.1, R6.2, TRIGGER.1, U1.GND1, U1.GND2; no longer 3/5V.2, C1.2, C10.2, C14.-, C2.2, C7.2, C8.2, C9.2, IC1.GND@1, IC1.GND@2, IC1.GND_PAD, J4.1, J5.1, JP1.1, JP12.2, JP14.2, JP7.1, PWR_LED.C, R10.2, R16.CW, R18.1, R19.1, R20.2, R7.1
- net MS1: no longer IC1.MS1, JP13.2, JP6.2, R1.1
- net MS2: no longer IC1.MS2, JP10.1, JP11.1, R2.1
- net MS3: no longer IC1.MS3, JP10.2, JP11.2, R3.1
- net N$1: now also J2.3, JP17.1; no longer D1.A, JP1.2, JP7.2
- net N$13: now also J1.4, R6.1, TRIGGER.2; no longer J6.2
- net N$14: now also C2.2, J1.8, R2.2; no longer J4.2
- net N$15: now also C1.2, J1.7, R1.2; no longer J5.2
- net N$16: now also S2.2; no longer S1.P1
- net N$2: now also C4.2, J1.6, R4.2, U1.D11; no longer PWR_LED.A, R9.1
- net N$3: now also J2.1, JP17.2; no longer R13.2, R16.CCW
- net N$6: now also C3.2, J1.5, R3.2, U1.D9; no longer IC2.ADJ, R6.2, R8.1
- net N$7: now also C5.2, J1.3, R5.2, U1.D12; no longer IC1.NC@2, U$4.P$1
- net N$8: now also J1.1, S2.1, U1.A1; no longer C6.1, IC1.CP1
- net RESET: no longer IC1.RESET, JP10.3, JP11.3, R5.1
- net SLEEP: no longer IC1.SLEEP, JP10.4, JP11.4, R4.1
- net STEP_IN: no longer JP12.3, JP14.3, R15.1
- net VCC: now also J1.2, S2.4; no longer APWR.2, C2.1, C7.1, IC1.VDD, JP12.1, JP14.1, R1.2, R11.2, R12.2, R13.1, R2.2, R3.2, R4.2, R5.2, R9.2, S1.S1
Other:
- note removed: "-moved vias and retraced as necessary on VCC and TOP layers"
- note removed: "-ran all traces directly away from IC"
- note removed: "-updated footprint for driver IC (1:1)"
- note removed: ".100" Headers"
- note removed: "3.5mm Screw Terminals"
- note removed: "3/5V Closed -> Vcc = 3.3V"
- note removed: "3/5V Normally Open -> Vcc=5.0V"
- note removed: "8V to 35V DC"
- note removed: "A rising edge on STEP"
- note removed: "APWR Normally Shorted"
- note removed: "Added current limiting resistors to STEP and DIR"
- note removed: "An easy to use bipolar stepper motor driver"
- note removed: "Be rated for >=50V"
- note removed: "Bi-polar Stepper Motor Outputs"
- note removed: "BigEasyDriver v1.6a"
- note removed: "Both C14 and C1 must"
- note removed: "Both take 0V to Vcc"
- note removed: "Brian Schmalz"
- note removed: "COILA+ and COILA-"
- note removed: "COILB+ and COILB-"
- note removed: "Change List:"
- note removed: "Changed R13 to 8.2K to improve range of current adjust pot"
- note removed: "Changed license from CC by 3.0 to CC by-sa 3.0"
- note removed: "Coil A of motor across"
- note removed: "Coil B of motor across"
- note removed: "Current adjust pot: adjusts max coil current. R13 set such that: At VCC = 3.3V, full clockwise = 2.08A coil current At VCC = 5V, 64% clockwise = 2.0A coil current Note driver can only output 2A coil current, and is dependent on input voltage, motor, and heat sinking/fan to reach this."
- note removed: "Cut to use your own"
- note removed: "D.N.I"
- note removed: "DEFAULT OPTIONS"
- note removed: "DIR is level sensitive"
- note removed: "Defaults to 5V for Vcc (logic supply), settable to 3.3V"
- note removed: "Do not connect or disconnect motor"
- note removed: "ENABLE = GND (enabled)"
- note removed: "For 35V V+ input"
- note removed: "From 0mA/phase to over 2A/phase"
- note removed: "MS1 = Vcc (1/16 microstep)"
- note removed: "MS2 = Vcc (1/16 microstep)"
- note removed: "MS3 = Vcc (1/16 microstep)"
- note removed: "Must use LM317"
- note removed: "NOTE: VCC is normally an OUTPUT. You do not need to"
- note removed: "Power Input JP1, JP7"
- note removed: "Produced by SparkFun Electronics"
- note removed: "RESET = Vcc (not reset)"
- note removed: "Removed large hole in solder mask on bottom"
- note removed: "Revised by Patrick Alberts"
- note removed: "SLEEP = Vcc (awake)"
- note removed: "Short JP10, or JP6 pins"
- note removed: "SparkFun design rules applied - minor layout tweaks, R13 now 2.49K"
- note removed: "Supply 8V to 35V DC power input on JP1 or JP7"
- note removed: "The only power needed is through M+ (motor power)."
- note removed: "The rest you can use, if you want"
- note removed: "Updated to standard 0603 foorprints, some rerouting, schematic nets changed"
- note removed: "Use 4 wire, 6 wire or 8 wire steper motors"
- note removed: "Vcc source from JP14 VCC"
- note removed: "Voltage regulator can supply 100mA"
- note removed: "You only need to connect M+, GND, STEP, DIR and the motor outputs. All other I/O is set to default to 1/16th microstep mode, and connections are not required for basic operation."
- note removed: "causes a step"
- note removed: "from the VCC pin."
- note removed: "only 15mA of which the BED needs."
- note removed: "supply power to the Big Easy Driver through VCC."
- note removed: "to GND or Vcc to override"
- note removed: "v1.0 BPS Origonal version"
- note removed: "v1.1 BPS Added pull-ups, re-routed"
- note removed: "v1.2 5/2/11 BPS Silk screen corrections, sense resistors now .11 ohms"
- note removed: "v1.3 SF 1/10/12"
- note removed: "v1.4 SF 4/17/2013 Fixed current adjustment pot silk so directions are correct"
- note removed: "v1.5 SF 6/27/2013"
- note removed: "v1.6 BPS 3/28/2014"
- note removed: "v16a"
- note removed: "while BigEasyDriver is powered"
- note removed: "www.schmalzhaus.com/BigEasyDriver"

Commit message: Updated top silk, removed some layout corners and increased version to 1.2.
Other:
- moved on the sheet: J1, J2, JP16, JP17, JP2, JP4, MOTOR, R1, R17, R2, R3, R4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
